Commit message: changes to xacro for compatability with ur5 macro

File: urdf/rg6_gripper.xacro (robot description, xacro)
@@ -1,7 +1,7 @@
 <?xml version="1.0" ?>
 <robot name="rg6" xmlns:xacro="http://www.ros.org/wiki/xacro">
-<xacro:include filename="$(find rg6_gripper_description)/urdf/materials.xacro" />
-<xacro:include filename="$(find rg6_gripper_description)/urdf/rg6_gripper.trans" />
-<xacro:include filename="$(find rg6_gripper_description)/urdf/rg6_gripper.gazebo" />
+<xacro:include filename="$(find rg6_gripper)/urdf/materials.xacro" />
+<xacro:include filename="$(find rg6_gripper)/urdf/rg6_gripper.trans" />
+<xacro:include filename="$(find rg6_gripper)/urdf/rg6_gripper.gazebo" />
 <link name="base_link">
   <inertial>
@@ -13,5 +13,5 @@
     <origin xyz="0 0 0" rpy="0 0 0"/>
     <geometry>
-      <mesh filename="package://rg6_gripper_description/meshes/base_link.stl" scale="0.001 0.001 0.001"/>
+      <mesh filename="package://rg6_gripper/meshes/base_link.stl" scale="0.001 0.001 0.001"/>
     </geometry>
     <material name="silver"/>
@@ -20,5 +20,5 @@
     <origin xyz="0 0 0" rpy="0 0 0"/>
     <geometry>
-      <mesh filename="package://rg6_gripper_description/meshes/base_link.stl" scale="0.001 0.001 0.001"/>
+      <mesh filename="package://rg6_gripper/meshes/base_link.stl" scale="0.001 0.001 0.001"/>
     </geometry>
   </collision>
@@ -33,5 +33,5 @@
     <origin xyz="0.031849 -1e-06 -0.04953" rpy="0 0 0"/>
     <geometry>
-      <mesh filename="package://rg6_gripper_description/meshes/g_main.stl" scale="0.001 0.001 0.001"/>
+      <mesh filename="package://rg6_gripper/meshes/g_main.stl" scale="0.001 0.001 0.001"/>
     </geometry>
     <material name="silver"/>
@@ -40,5 +40,5 @@
     <origin xyz="0.031849 -1e-06 -0.04953" rpy="0 0 0"/>
     <geometry>
-      <mesh filename="package://rg6_gripper_description/meshes/g_main.stl" scale="0.001 0.001 0.001"/>
+      <mesh filename="package://rg6_gripper/meshes/g_main.stl" scale="0.001 0.001 0.001"/>
     </geometry>
   </collision>
@@ -53,5 +53,5 @@
     <origin xyz="-0.023851 -0.012801 -0.13453" rpy="0 0 0"/>
     <geometry>
-      <mesh filename="package://rg6_gripper_description/meshes/l_out.stl" scale="0.001 0.001 0.001"/>
+      <mesh filename="package://rg6_gripper/meshes/l_out.stl" scale="0.001 0.001 0.001"/>
     </geometry>
     <material name="silver"/>
@@ -60,5 +60,5 @@
     <origin xyz="-0.023851 -0.012801 -0.13453" rpy="0 0 0"/>
     <geometry>
-      <mesh filename="package://rg6_gripper_description/meshes/l_out.stl" scale="0.001 0.001 0.001"/>
+      <mesh filename="package://rg6_gripper/meshes/l_out.stl" scale="0.001 0.001 0.001"/>
     </geometry>
   </collision>
@@ -73,5 +73,5 @@
     <origin xyz="0.023749 -0.012801 -0.13453" rpy="0 0 0"/>
     <geometry>
-      <mesh filename="package://rg6_gripper_description/meshes/r_out.stl" scale="0.001 0.001 0.001"/>
+      <mesh filename="package://rg6_gripper/meshes/r_out.stl" scale="0.001 0.001 0.001"/>
     </geometry>
     <material name="silver"/>
@@ -80,5 +80,5 @@
     <origin xyz="0.023749 -0.012801 -0.13453" rpy="0 0 0"/>
     <geometry>
-      <mesh filename="package://rg6_gripper_description/meshes/r_out.stl" scale="0.001 0.001 0.001"/>
+      <mesh filename="package://rg6_gripper/meshes/r_out.stl" scale="0.001 0.001 0.001"/>
     </geometry>
   </collision>
@@ -93,5 +93,5 @@
     <origin xyz="-0.071235 0.012499 -0.19895" rpy="0 0 0"/>
     <geometry>
-      <mesh filename="package://rg6_gripper_description/meshes/l_tip.stl" scale="0.001 0.001 0.001"/>
+      <mesh filename="package://rg6_gripper/meshes/l_tip.stl" scale="0.001 0.001 0.001"/>
     </geometry>
     <material name="silver"/>
@@ -100,5 +100,5 @@
     <origin xyz="-0.071235 0.012499 -0.19895" rpy="0 0 0"/>
     <geometry>
-      <mesh filename="package://rg6_gripper_description/meshes/l_tip.stl" scale="0.001 0.001 0.001"/>
+      <mesh filename="package://rg6_gripper/meshes/l_tip.stl" scale="0.001 0.001 0.001"/>
     </geometry>
   </collision>
@@ -113,5 +113,5 @@
     <origin xyz="0.071133 0.012499 -0.199024" rpy="0 0 0"/>
     <geometry>
-      <mesh filename="package://rg6_gripper_description/meshes/r_tip.stl" scale="0.001 0.001 0.001"/>
+      <mesh filename="package://rg6_gripper/meshes/r_tip.stl" scale="0.001 0.001 0.001"/>
     </geometry>
     <material name="silver"/>
@@ -120,5 +120,5 @@
     <origin xyz="0.071133 0.012499 -0.199024" rpy="0 0 0"/>
     <geometry>
-      <mesh filename="package://rg6_gripper_description/meshes/r_tip.stl" scale="0.001 0.001 0.001"/>
+      <mesh filename="package://rg6_gripper/meshes/r_tip.stl" scale="0.001 0.001 0.001"/>
     </geometry>
   </collision>
@@ -133,5 +133,5 @@
     <origin xyz="-0.010551 -0.000101 -0.15763" rpy="0 0 0"/>
     <geometry>
-      <mesh filename="package://rg6_gripper_description/meshes/l_inner.stl" scale="0.001 0.001 0.001"/>
+      <mesh filename="package://rg6_gripper/meshes/l_inner.stl" scale="0.001 0.001 0.001"/>
     </geometry>
     <material name="silver"/>
@@ -140,5 +140,5 @@
     <origin xyz="-0.010551 -0.000101 -0.15763" rpy="0 0 0"/>
     <geometry>
-      <mesh filename="package://rg6_gripper_description/meshes/l_inner.stl" scale="0.001 0.001 0.001"/>
+      <mesh filename="package://rg6_gripper/meshes/l_inner.stl" scale="0.001 0.001 0.001"/>
     </geometry>
   </collision>
@@ -153,5 +153,5 @@
     <origin xyz="0.010449 -0.000101 -0.15763" rpy="0 0 0"/>
     <geometry>
-      <mesh filename="package://rg6_gripper_description/meshes/r_inner.stl" scale="0.001 0.001 0.001"/>
+      <mesh filename="package://rg6_gripper/meshes/r_inner.stl" scale="0.001 0.001 0.001"/>
     </geometry>
     <material name="silver"/>
@@ -160,5 +160,5 @@
     <origin xyz="0.010449 -0.000101 -0.15763" rpy="0 0 0"/>
     <geometry>
-      <mesh filename="package://rg6_gripper_description/meshes/r_inner.stl" scale="0.001 0.001 0.001"/>
+      <mesh filename="package://rg6_gripper/meshes/r_inner.stl" scale="0.001 0.001 0.001"/>
     </geometry>
   </collision>
